File: flight computer/flight computer.kicad_sch (KiCad schematic)
At the start: 94 parts, among them IC1 114993390, IC2 ADXL375BCCZ-RL, J1 SMA-J-P-H-ST-EM1, J2 SMA-J-P-H-ST-EM1, J3 Micro_SD_Card, J4 USB_C_Receptacle_USB2.0_16P, Q1 BSS138, Q2 BSS84, Q3 PMOS, Q4 NMOS, Q5 PMOS, U1 TPS56A37RPAR, U10 SIA440DJ-T1-GE3, U11 high, U12 medium, U13 low, U14 power, U15 fault, U16 JS207011SCQNR, U2 BMP581, U3 BNO086, U4 BTM9011EP, U5 RP2354B, U6 MAX-M10S-00B, U7 AZ1117CH-3.3TRG1, U8 VND9025AJTR, U9 74LVC1G07GW_125

Commit message: Organising the schematic
Parts:
- removed C1, C2, C22: 10uF, Capacitor_SMD:C_1206_3216Metric_Pad1.33x1.80mm_HandSolder, symbol Device:C
- removed C10, C11, C12, C13, C15, C16, C25, C26, C27, C28, C3, C5, C9: 0.1uF, Capacitor_SMD:C_0805_2012Metric_Pad1.18x1.45mm_HandSolder, symbol Device:C
- removed C14: 1nF, Capacitor_SMD:C_0805_2012Metric_Pad1.18x1.45mm_HandSolder, symbol Device:C
- removed C17: 560uF, Capacitor_SMD:C_0805_2012Metric_Pad1.18x1.45mm_HandSolder, symbol Device:C
- removed C18, C20, C21: 10nF, Capacitor_SMD:C_0805_2012Metric_Pad1.18x1.45mm_HandSolder, symbol Device:C
- removed C19: 47pF, Capacitor_SMD:C_0805_2012Metric_Pad1.18x1.45mm_HandSolder, symbol Device:C
- removed C23, C7, C8: 22uF, Capacitor_SMD:C_1210_3225Metric_Pad1.33x2.70mm_HandSolder, symbol Device:C
- removed C24: 0.1uF, symbol Device:C
- removed C4: 47nF, Capacitor_SMD:C_0805_2012Metric_Pad1.18x1.45mm_HandSolder, symbol Device:C
- removed C6: 150pF, Capacitor_SMD:C_0805_2012Metric_Pad1.18x1.45mm_HandSolder, symbol Device:C
- removed CR1: SMBJ15A, Snapeda:DO-214AASMB_J-BEND_LTF-L, symbol Snapeda:SMBJ15A
- removed D1: 8.6V, symbol Device:D_Zener
- removed D2, D3, D6: D_Schottky, symbol Device:D_Schottky
- removed D4: D, symbol Device:D
- removed D5: D_Zener, symbol Device:D_Zener
- removed IC1: 114993390, Samacsys:114993390, symbol Samacsys:114993390
- removed IC2: ADXL375BCCZ-RL, Samacsys:ADXL375BCCZRL, symbol Samacsys:ADXL375BCCZ-RL
- removed J1, J2: SMA-J-P-H-ST-EM1, Snapeda:SAMTEC_SMA-J-P-H-ST-EM1, symbol Snapeda:SMA-J-P-H-ST-EM1
- removed J3: Micro_SD_Card, Connector_Card:microSD_HC_Molex_47219-2001, symbol Connector:Micro_SD_Card
- removed J4: USB_C_Receptacle_USB2.0_16P, Connector_USB:USB_C_Receptacle_GCT_USB4105-xx-A_16P_TopMnt_Horizontal, symbol Connector:USB_C_Receptacle_USB2.0_16P
- removed L1: 3.3uH, Snapeda:IND_SRP1265A-3R3M, symbol Device:L_Iron
- removed L2, L3: 27uH, Inductor_SMD:L_0805_2012Metric_Pad1.05x1.20mm_HandSolder, symbol Device:L
- removed LS1: CPT-1203-78-SMT-TR, Snapeda:XDCR_CPT-1203-78-SMT-TR, symbol Snapeda:CPT-1203-78-SMT-TR
- removed Q1: BSS138, Package_TO_SOT_SMD:SOT-23-3, symbol Simulation_SPICE:NMOS
- removed Q2: BSS84, Package_TO_SOT_SMD:SOT-23-3, symbol Simulation_SPICE:PMOS
- removed Q3, Q5: PMOS, symbol Simulation_SPICE:PMOS
- removed Q4: NMOS, symbol Simulation_SPICE:NMOS
- removed R1, R2, R4, R7, R8, R9: 10k, Resistor_SMD:R_0805_2012Metric_Pad1.20x1.40mm_HandSolder, symbol Device:R
- removed R10: 820, Resistor_SMD:R_0805_2012Metric_Pad1.20x1.40mm_HandSolder, symbol Device:R
- removed R11: 100k, Resistor_SMD:R_0805_2012Metric_Pad1.20x1.40mm_HandSolder, symbol Device:R
- removed R12: 10, Resistor_SMD:R_0805_2012Metric_Pad1.20x1.40mm_HandSolder, symbol Device:R
- removed R13, R14, R18: 100k, symbol Device:R
- removed R15: 1M, symbol Device:R
- removed R16, R28: 330, symbol Device:R
- removed R17: 4.7k, symbol Device:R
- removed R19, R20: 5.1k, symbol Device:R
- removed R21, R22, R23, R24, R25, R26, R27: 110, symbol Device:R
- removed R3: 52.3k, Resistor_SMD:R_0805_2012Metric_Pad1.20x1.40mm_HandSolder, symbol Device:R
- removed R5: 49.9, Resistor_SMD:R_0805_2012Metric_Pad1.20x1.40mm_HandSolder, symbol Device:R
- removed R6: 73.2k, Resistor_SMD:R_0805_2012Metric_Pad1.20x1.40mm_HandSolder, symbol Device:R
- removed U1: TPS56A37RPAR, Snapeda:RPA0010A-MFG, symbol Snapeda:TPS56A37RPAR
- removed U10: SIA440DJ-T1-GE3, Snapeda:SON_1DJ-T1-GE3_VIS, symbol Snapeda:SIA440DJ-T1-GE3
- removed U11: high, Snapeda:LTST-BILED-15X16, symbol Snapeda:LTST-C195KGJRKT
- removed U12: medium, Snapeda:LTST-BILED-15X16, symbol Snapeda:LTST-C195KGJRKT
- removed U13: low, Snapeda:LTST-BILED-15X16, symbol Snapeda:LTST-C195KGJRKT
- removed U14: power, Snapeda:LTST-BILED-15X16, symbol Snapeda:LTST-C195KGJRKT
- removed U15: fault, Snapeda:LTST-BILED-15X16, symbol Snapeda:LTST-C195KGJRKT
- removed U16: JS207011SCQNR, Snapeda:SOIC_SCQNR_CNK, symbol Snapeda:JS207011SCQNR
- removed U2: BMP581, Snapeda:QFN10_BMP581_BOS-L, symbol Snapeda:BMP581
- removed U3: BNO086, Snapeda:IC_BNO086, symbol Snapeda:BNO086
- removed U4: BTM9011EP, Samacsys:SOP65P600X115-15N, symbol Samacsys:BTM9011EP
- removed U5: RP2354B, Package_DFN_QFN:QFN-80-1EP_10x10mm_P0.4mm_EP3.4x3.4mm, symbol MCU_RaspberryPi:RP2354B
- removed U6: MAX-M10S-00B, Snapeda:XCVR_MAX-M10S-00B, symbol Snapeda:MAX-M10S-00B
- removed U7: AZ1117CH-3.3TRG1, Snapeda:SOT-223_DIO-L, symbol Snapeda:AZ1117CH-3.3TRG1
- removed U8: VND9025AJTR, Snapeda:IC_POWERSSO-16_STM-L, symbol Snapeda:VND9025AJTR
- removed U9: 74LVC1G07GW_125, Snapeda:IC_74LVC1G07GW_125, symbol Snapeda:74LVC1G07GW_125
- added C45, C46, C48, C49, C62, C63, C64, C65, C66, C67, C68, C73: 0.1uF, Capacitor_SMD:C_0805_2012Metric_Pad1.18x1.45mm_HandSolder, symbol Device:C
- added C69, C70, C71, C72, C74: 4.7uF, Capacitor_SMD:C_0805_2012Metric_Pad1.18x1.45mm_HandSolder, symbol Device:C
- added C75, C76: 27pF, Capacitor_SMD:C_0805_2012Metric_Pad1.18x1.45mm_HandSolder, symbol Device:C
- added IC1: AT25SF128A-SHB-T, Samacsys:SOIC127P798X216-8N, symbol Samacsys:AT25SF128A-SHB-T
- added L1: 3.3uH, Snapeda:IND_SRP1265A-3R3M, symbol Device:L
- added R49: 33, Resistor_SMD:R_0805_2012Metric_Pad1.20x1.40mm_HandSolder, symbol Device:R
- added R64, R65: 27, Resistor_SMD:R_0805_2012Metric_Pad1.20x1.40mm_HandSolder, symbol Device:R
- added R66, R67, R68: 1k, Resistor_SMD:R_0805_2012Metric_Pad1.20x1.40mm_HandSolder, symbol Device:R
- added SW3, SW4: PTS636SL43SMTRLFS, Snapeda:SW_PTS636S-J_CNK, symbol Snapeda:PTS636SL43SMTRLFS
- added U6: RP2350B, Snapeda:IC_BNO086, symbol MCU_RaspberryPi:RP2350B
- added Y1: ABM8G-12.000MHZ-18-D2Y-T, Snapeda:CRYSTAL_ABM8G_ABR-L, symbol Snapeda:ABM8G-12.000MHZ-18-D2Y-T
Connections:
- net +3.3V: now also C45.1, C46.1, C48.1, C49.1, C62.1, C63.1, C64.1, C65.1, C66.1, C71.1, C73.1, C74.1, IC1.8 (VCC), R49.2, U6.15 (IOVDD), U6.24 (IOVDD), U6.29 (IOVDD), U6.41 (IOVDD), U6.5 (IOVDD), U6.50 (IOVDD), U6.59 (ADC_AVDD), U6.60 (IOVDD), U6.64 (VREG_VIN), U6.68 (USB_OTP_VDD), U6.69 (QSPI_IOVDD), U6.76 (IOVDD)
- net ADXL375 CS: now also U6.2 (GPIO5)
- net BMP581 CS: now also U6.3 (GPIO6)
- net BNO086 CS: now also U6.4 (GPIO7)
- net BTM9011EP CS: now also U6.80 (GPIO3)
- net BTM9011EP IS: now also U6.56 (GPIO45/ADC5)
- net GND: now also C45.2, C46.2, C48.2, C49.2, C62.2, C63.2, C64.2, C65.2, C66.2, C67.2, C68.2, C69.2, C70.2, C71.2, C72.2, C73.2, C74.2, C75.1, C76.1, IC1.4 (GND), R68.2, SW4.2, U6.62 (VREG_PGND), U6.81 (GND), Y1.2, Y1.4
- net LED fault: now also U6.42 (GPIO33)
- net LED high green: now also U6.28 (GPIO27)
- net LED high red: now also U6.36 (GPIO28)
- net LED low green: now also U6.39 (GPIO31)
- net LED low red: now also U6.40 (GPIO32)
- net LED medium green: now also U6.37 (GPIO29)
- net LED medium red: now also U6.38 (GPIO30)
- net MISO: now also U6.77 (GPIO0)
- net MOSI: now also U6.78 (GPIO1)
- net SCK: now also U6.79 (GPIO2)
- net SD CLK: now also U6.43 (GPIO34)
- net SD CMD: now also U6.44 (GPIO35)
- net SD DAT0: now also U6.45 (GPIO36)
- net SD DAT1: now also U6.46 (GPIO37)
- net SD DAT2: now also U6.47 (GPIO38)
- net SD DAT3: now also U6.48 (GPIO39)
- net SX1262 CS: now also U6.1 (GPIO4)
- net VND9025 IN0: now also U6.6 (GPIO8)
- net VND9025 IN1: now also U6.7 (GPIO9)
- net buzzer: now also U6.9 (GPIO11)
- net power signal: now also U6.55 (GPIO44/ADC4)
- new net: C70.1, R49.1, U6.61 (VREG_AVDD)
- new net: R68.1, SW3.2
- new net: R65.1, U6.67 (USB_DP)
- new net: SW3.1, U6.35 (RUN)
- new net: C75.2, R66.2, Y1.3
- new net: L1.2, U6.63 (VREG_LX)
- new net: R64.1, U6.66 (USB_DM)
- new net: R67.2, SW4.1
- new net +1.1V: C67.1, C68.1, C69.1, C72.1, L1.1, U6.10 (DVDD), U6.32 (DVDD), U6.51 (DVDD), U6.65 (VREG_FB)
- new net QSPI_SCLK: IC1.6 (SCK), U6.71 (QSPI_SCLK)
- new net QSPI_SD0: IC1.5 (SI_(I/O0)), U6.72 (QSPI_SD0)
- new net QSPI_SD1: IC1.2 (SO_(I/O1)), U6.74 (QSPI_SD1)
- new net QSPI_SD2: IC1.3 (~{WP_(I}/O2)), U6.73 (QSPI_SD2)
- new net QSPI_SD3: IC1.7 (~{HOLD_(I}/O3)), U6.70 (QSPI_SD3)
- new net QSPI_SS: IC1.1 (~{CS}), R67.1, U6.75 (~{QSPI_SS})
- new net USB_DM: R64.2
- new net USB_DP: R65.2
- new net VND9025 fault: U6.8 (GPIO10)
- new net XIN: C76.2, U6.30 (XIN), Y1.1
- new net XOUT: R66.1, U6.31 (XOUT)
- new net motor in a: U6.57 (GPIO46/ADC6)
- new net motor in b: U6.58 (GPIO47/ADC7)
- new net pyro 1 continuity: U6.49 (GPIO40/ADC0)
- new net pyro 1 gate: U6.13 (GPIO14)
- new net pyro 2 continuity: U6.52 (GPIO41/ADC1)
- new net pyro 2 gate: U6.14 (GPIO15)
- new net pyro 3 continuity: U6.53 (GPIO42/ADC2)
- new net pyro 3 gate: U6.16 (GPIO16)
- new net pyro 4 continuity: U6.54 (GPIO43/ADC3)
- new net pyro 4 gate: U6.17 (GPIO17)
- new net servo PWM 1: U6.11 (GPIO12)
- new net servo PWM 2: U6.12 (GPIO13)
- new net servo PWM 3: U6.18 (GPIO18)
- new net servo PWM 4: U6.19 (GPIO19)
- no-connect marks 28 -> 2

Commit message: Finalisation of Schematic
Parts:
- removed SW3, SW4: PTS636SL43SMTRLFS, Snapeda:SW_PTS636S-J_CNK, symbol Snapeda:PTS636SL43SMTRLFS
- added J1: JST, Connector_PinHeader_2.54mm:PinHeader_1x03_P2.54mm_Vertical_SMD_Pin1Right, symbol Connector:Conn_01x03_Pin
- added S1, S2: PTS647SM38SMTR2_LFS, Samacsys:PTS647SM38SMTR2LFS, symbol Samacsys:PTS647SM38SMTR2_LFS
- IC1: footprint Samacsys:SOIC127P798X216-8N -> Snapeda:IC8_AT25SF128A-SHB-T_ADO-L
- L1: footprint Snapeda:IND_SRP1265A-3R3M -> Snapeda:IND_TAIYO_NRS4018_TAY
- U1: renamed from U6; footprint Snapeda:IC_BNO086 -> Package_DFN_QFN:QFN-80-1EP_10x10mm_P0.4mm_EP3.4x3.4mm
- renumbered C71 to C1, C49 to C10, C62 to C11, C63 to C12, C64 to C13, C65 to C14, C66 to C15, C76 to C16, C75 to C17, C73 to C18, C74 to C19, C72 to C2, C69 to C3, C70 to C4, C68 to C5, C67 to C6, C45 to C7, C46 to C8, C48 to C9, R68 to R1, R67 to R2, R49 to R3, R64 to R4, R65 to R5, R66 to R6
Connections:
- net LED low green is gone; now on net ADXL375 CS: U1.39 (GPIO31)
- net LED medium red is gone; now on net BNO086 CS: U1.38 (GPIO30)
- net buzzer is gone; now on net motor in b: U1.9 (GPIO11)
- net ADXL375 CS: no longer U1.2 (GPIO5)
- net BMP581 CS: now also U1.80 (GPIO3); no longer U1.3 (GPIO6)
- net BNO086 CS: no longer U1.4 (GPIO7)
- net BTM9011EP CS: now also U1.55 (GPIO44/ADC4); no longer U1.80 (GPIO3)
- net GND: now also J1.2 (Pin_2), S1.3 (COM_1), S1.4 (COM_2)
- net SX1262 CS: now also U1.26 (GPIO25); no longer U1.1 (GPIO4)
- net VND9025 IN0: now also U1.20 (GPIO20); no longer U1.6 (GPIO8)
- net VND9025 IN1: now also U1.22 (GPIO22); no longer U1.7 (GPIO9)
- net VND9025 fault: now also U1.21 (GPIO21); no longer U1.8 (GPIO10)
- net motor in a: now also U1.8 (GPIO10); no longer U1.57 (GPIO46/ADC6)
- net motor in b: no longer U1.58 (GPIO47/ADC7)
- net power controller: now also U1.58 (GPIO47/ADC7)
- net power signal: now also U1.57 (GPIO46/ADC6); no longer U1.55 (GPIO44/ADC4)
- net at R1.1: now also S2.3 (COM_1), S2.4 (COM_2)
- net at U1.35 (RUN): now also S2.1 (NO_1), S2.2 (NO_2)
- net SX1262 rf switch: now reaches U1.23 (GPIO23)
- net SX1262 reset: now reaches U1.25 (GPIO24)
- net SX1262 busy: now reaches U1.27 (GPIO26)
- net SWCLK: now reaches U1.33 (SWCLK)
- net SWCLK: now also J1.1 (Pin_1)
- net SWDIO: now reaches U1.34 (SWDIO)
- net SWDIO: now also J1.3 (Pin_3)
- net at R2.2: now also S1.1 (NO_1), S1.2 (NO_2)
- net LED fault renamed pin out 2
- net LED high green renamed SX1262 int
- net LED high red renamed BNO086 wake
- net LED low red renamed pin out 1
- net LED medium green renamed BNO086 int
- new net MAX M10S RX: U1.2 (GPIO5)
- new net MAX M10S TX: U1.1 (GPIO4)
- new net MAX M10S boot: U1.7 (GPIO9)
- new net MAX M10S int: U1.4 (GPIO7)
- new net MAX M10S reset: U1.6 (GPIO8)
- new net MAX M10S timepulse: U1.3 (GPIO6)
- no-connect marks 2 -> 0
Other:
- note added: "JST debug header"
- note added: "crystal"
- note added: "flash"
- note added: "microcontroller"
- title: (none) -> microcontroller
- moved on the sheet: C1, C10, C11, C12, C13, C14, C15, C16, C17, C18, C19, C2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
