File: flight computer/interfaces.kicad_sch (KiCad schematic)
At the start: 22 parts, among them J14 USB_C_Receptacle_USB2.0_16P, J15 Micro_SD_Card, U1 LTST-C195KGJRKT, U2 LTST-C195KGJRKT, U3 LTST-C195KGJRKT, U4 LTST-C195KGJRKT, U5 LTST-C195KGJRKT

Commit message: Finalisation of Schematic
Parts:
- removed C42: 2.2uF, Capacitor_SMD:C_0805_2012Metric_Pad1.18x1.45mm_HandSolder, symbol Device:C
- removed C43: 0.1uF, Capacitor_SMD:C_0805_2012Metric_Pad1.18x1.45mm_HandSolder, symbol Device:C
- removed J15: Micro_SD_Card, Connector_Card:microSD_HC_Molex_47219-2001, symbol Connector:Micro_SD_Card
- removed LS2: CPT-1203-78-SMT-TR, Snapeda:XDCR_CPT-1203-78-SMT-TR, symbol Snapeda:CPT-1203-78-SMT-TR
- removed R43, R44, R45, R46, R47, R48, R50, R62: 110, Resistor_SMD:R_0805_2012Metric_Pad1.20x1.40mm_HandSolder, symbol Device:R
- removed R55: 1k, Resistor_SMD:R_0805_2012Metric_Pad1.20x1.40mm_HandSolder, symbol Device:R
- removed U1: LTST-C195KGJRKT, Snapeda:SOIC_SCQNR_CNK, symbol Snapeda:LTST-C195KGJRKT
- removed U2: LTST-C195KGJRKT, Snapeda:IC_POWERSSO-16_STM-L, symbol Snapeda:LTST-C195KGJRKT
- removed U3: LTST-C195KGJRKT, Snapeda:RPA0010A-MFG, symbol Snapeda:LTST-C195KGJRKT
- removed U4: LTST-C195KGJRKT, Snapeda:POWERPAK-1212-8S_VIS, symbol Snapeda:LTST-C195KGJRKT
- removed U5: LTST-C195KGJRKT, Snapeda:SOT-223_DIO-L, symbol Snapeda:LTST-C195KGJRKT
- added C32, C33, C34, C35, C37: 0.1uF, Capacitor_SMD:C_0805_2012Metric_Pad1.18x1.45mm_HandSolder, symbol Device:C
- added C36: 4.7uF, Capacitor_SMD:C_0805_2012Metric_Pad1.18x1.45mm_HandSolder, symbol Device:C
- added H1, H2, H3, H4: MountingHole, MountingHole:MountingHole_3.2mm_M3, symbol Mechanical:MountingHole
- added J10: Micro_SD_Card, Connector_Card:microSD_HC_Molex_47219-2001, symbol Connector:Micro_SD_Card
- added J9: GPIO, Samacsys:5452257, symbol Samacsys:5452257
- added LED1, LED2, LED3, LED4: COM-16347, Snapeda:COM-16347_SPK-L, symbol Snapeda:COM-16347
- added LS1: CPT-1203-78-SMT-TR, Snapeda:XDCR_CPT-1203-78-SMT-TR, symbol Snapeda:CPT-1203-78-SMT-TR
- added R17, R20, R21: 1k, Resistor_SMD:R_0805_2012Metric_Pad1.20x1.40mm_HandSolder, symbol Device:R
- D5: renamed from D10; footprint (none) -> Diode_SMD:D_SOD-123
- R18: renamed from R24; footprint (none) -> Resistor_SMD:R_0805_2012Metric_Pad1.20x1.40mm_HandSolder
- R19: renamed from R25; footprint (none) -> Resistor_SMD:R_0805_2012Metric_Pad1.20x1.40mm_HandSolder
- renumbered J14 to J8
Connections:
- net +3.3V: now also C36.1, C37.1, J10.4 (VDD)
- net +5V: now also C32.1, C33.1, C34.1, C35.1, LED1.1 (VDD), LED2.1 (VDD), LED3.1 (VDD), LED4.1 (VDD)
- net GND: now also C32.2, C33.2, C34.2, C35.2, C36.2, C37.2, J10.6 (VSS), J10.SH (SHIELD), LED1.3 (VSS), LED2.3 (VSS), LED3.3 (VSS), LED4.3 (VSS), LS1.2
- net SD CLK: now also J10.5 (CLK)
- net SD CMD: now also J10.3 (CMD)
- net SD DAT0: now also J10.7 (DAT0)
- net SD DAT1: now also J10.8 (DAT1)
- net SD DAT2: now also J10.1 (DAT2)
- net SD DAT3: now also J10.2 (DAT3/CD)
- net buzzer: now also R17.2
- new net: LS1.1, R17.1
- new net: LED3.2 (DOUT), LED4.4 (DIN)
- new net: J9.1, R20.2
- new net: J9.2, R21.2
- new net: LED2.2 (DOUT), LED3.4 (DIN)
- new net: LED1.2 (DOUT), LED2.4 (DIN)
- new net LED controller: LED1.4 (DIN)
- new net pin out 1: R20.1
- new net pin out 2: R21.1
- no-connect marks 4 -> 3
Other:
- note added: "GPIO header"
- note added: "mounting holes"
- title: (none) -> ports & peripherials
