File: flight computer/power.kicad_sch (KiCad schematic)
At the start: 36 parts, among them J13 ED555/2DS, Q5 NMOS, Q6 PMOS, U17 SISS65DN-T1-GE3, U18 AZ1117CH-3.3TRG1, U19 JS207011SCQNR, U20 TPS56A37RPAR, U21 VND9025AJTR

Commit message: Finalisation of Schematic
Parts:
- removed D6: D, symbol Device:D
- removed J13: ED555/2DS, Snapeda:CONN_ED555&slash_2DS_OST, symbol Snapeda:ED555_2DS
- removed U19: JS207011SCQNR, Snapeda:SOIC_SCQNR_CNK, symbol Snapeda:JS207011SCQNR
- added D1: D_Schottky, Diode_SMD:D_SOD-123, symbol Device:D_Schottky
- added J2: battery in, Samacsys:5452257, symbol Samacsys:5452257
- added J3: battery sw, Samacsys:5452257, symbol Samacsys:5452257
- added J4: pyro sw, Samacsys:5452257, symbol Samacsys:5452257
- added J5: 12V out, Samacsys:5452257, symbol Samacsys:5452257
- added J6: 5V out, Samacsys:5452257, symbol Samacsys:5452257
- added J7: 3.3V out, Samacsys:5452257, symbol Samacsys:5452257
- added R23: 100k, Resistor_SMD:R_0805_2012Metric_Pad1.20x1.40mm_HandSolder, symbol Device:R
- added U6: JS207011SCQNR, Snapeda:SOIC_SCQNR_CNK, symbol Snapeda:JS207011SCQNR
- C27: renamed from C36; footprint (none) -> Capacitor_SMD:C_0805_2012Metric_Pad1.18x1.45mm_HandSolder
- D2: renamed from D7; footprint (none) -> Diode_SMD:D_SOD-123
- D3: renamed from D8; footprint (none) -> Diode_SMD:D_SOD-123
- D4: renamed from D9; footprint (none) -> Diode_SMD:D_SOD-123
- Q1: renamed from Q5; footprint (none) -> Package_TO_SOT_SMD:SOT-23-3
- Q2: renamed from Q6; footprint (none) -> Package_TO_SOT_SMD:SOT-23-3
- R11: renamed from R37; footprint (none) -> Resistor_SMD:R_0805_2012Metric_Pad1.20x1.40mm_HandSolder
- R12: renamed from R38; footprint (none) -> Resistor_SMD:R_0805_2012Metric_Pad1.20x1.40mm_HandSolder
- R16: renamed from R42; footprint (none) -> Resistor_SMD:R_0805_2012Metric_Pad1.20x1.40mm_HandSolder
- R7: renamed from R35; footprint (none) -> Resistor_SMD:R_0805_2012Metric_Pad1.20x1.40mm_HandSolder
- R9: renamed from R34; footprint (none) -> Resistor_SMD:R_0805_2012Metric_Pad1.20x1.40mm_HandSolder
- renumbered C30 to C20, C31 to C21, C32 to C22, C33 to C23, C34 to C24, C35 to C25, C41 to C26, C37 to C28, C38 to C29, C39 to C30, C40 to C31, CR2 to CR1, L4 to L2, R36 to R10, R39 to R13, R40 to R14, R41 to R15, R33 to R8, U21 to U2, U17 to U3, U18 to U4, U20 to U5
Connections:
- net +12V main: now also C27.1, Q2.3 (S), R12.1, J3.1
- net +12V pyro: now also J4.1
- net +3.3V: now also J7.1
- net +5V: now also J6.1, R23.2
- net +VBAT: now also J2.1
- net GND: now also D1.1 (K), J2.2, J5.2, J6.2, J7.2, U6.2, U6.3, U6.4, U6.6, U6.7, U6.8
- net at D2.1 (K), D3.1 (K): now also U6.1, U6.5
- net at R7.1, U2.4 (GND): now also D1.2 (A)
- net +12V power: now reaches D4.1 (K), Q2.1 (D)
- net +12V power: now also J3.2
- net at U5.4 (PG): now also R23.1
- net +12V motor renamed +12V I/O
- net +12V I/O: now also J5.1
- new net +12V pyro sw: J4.2
- no-connect marks 9 -> 4
Other:
- note added: "power headers"
- note removed: "battery header"
- title: (none) -> power management
- moved on the sheet: C20, C21, C26, C27, C29, C30, C31, CR1, D2, D3, D4, L2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
