File: flight computer/power.kicad_sch (KiCad schematic)
At the start: 42 parts, among them J2 battery in, J3 battery sw, J4 pyro sw, J5 12V out, J6 5V out, J7 3.3V out, Q1 NMOS, Q2 PMOS, U2 VND9025AJTR, U3 SISS65DN-T1-GE3, U4 AZ1117CH-3.3TRG1, U5 TPS56A37RPAR, U6 JS207011SCQNR

Commit message: General progress on the PCB
Parts:
- removed D2, D3: D_Schottky, Diode_SMD:D_SOD-123, symbol Device:D_Schottky
- removed Q1: NMOS, Package_TO_SOT_SMD:SOT-23-3, symbol Simulation_SPICE:NMOS
- removed R11: 200k, Resistor_SMD:R_0805_2012Metric_Pad1.20x1.40mm_HandSolder, symbol Device:R
- removed R9: 330, Resistor_SMD:R_0805_2012Metric_Pad1.20x1.40mm_HandSolder, symbol Device:R
- added R24, R25: 0, Resistor_SMD:R_0603_1608Metric_Pad0.98x0.95mm_HandSolder, symbol Device:R
- C20, C22, C23: footprint Capacitor_SMD:C_1206_3216Metric_Pad1.33x1.80mm_HandSolder -> Capacitor_SMD:C_1210_3225Metric_Pad1.33x2.70mm_HandSolder
- C24, C25, C26, C27, C28, C29: footprint Capacitor_SMD:C_0805_2012Metric_Pad1.18x1.45mm_HandSolder -> Capacitor_SMD:C_0603_1608Metric_Pad1.08x0.95mm_HandSolder
- R10, R12, R13, R14, R15, R16, R23, R7, R8: footprint Resistor_SMD:R_0805_2012Metric_Pad1.20x1.40mm_HandSolder -> Resistor_SMD:R_0603_1608Metric_Pad0.98x0.95mm_HandSolder
Connections:
- net +12V I/O: now also U2.13 (OUTPUT0), U2.14 (OUTPUT0), U2.15 (OUTPUT0), U2.16 (OUTPUT0); no longer U2.10 (OUTPUT1), U2.11 (OUTPUT1), U2.12 (OUTPUT1), U2.9 (OUTPUT1)
- net +12V pyro: now also U2.10 (OUTPUT1), U2.11 (OUTPUT1), U2.12 (OUTPUT1), U2.9 (OUTPUT1); no longer U2.13 (OUTPUT0), U2.14 (OUTPUT0), U2.15 (OUTPUT0), U2.16 (OUTPUT0)
- net at U6.1, U6.5: now also C27.2, Q2.2 (G), R12.2
- net at R13.1, R14.2: now also R24.1; no longer C29.2
- net at C28.2: now also R25.1; no longer U5.7 (BOOT)
- new net: R25.2, U5.7 (BOOT)
- new net: C29.2, R24.2
Other:
- moved on the sheet: C28, C29, C30, C31, J2, J3, J4, J5, J6, J7, L2, R13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

Commit message: Tried a more effective layout
Parts:
- removed C26, C27: 0.1uF, Capacitor_SMD:C_0603_1608Metric_Pad1.08x0.95mm_HandSolder, symbol Device:C
- removed D1: D_Schottky, Diode_SMD:D_SOD-123, symbol Device:D_Schottky
- removed Q2: PMOS, Package_TO_SOT_SMD:SOT-23-3, symbol Simulation_SPICE:PMOS
- removed R12: 100k, Resistor_SMD:R_0603_1608Metric_Pad0.98x0.95mm_HandSolder, symbol Device:R
- removed R7: 4.7k, Resistor_SMD:R_0603_1608Metric_Pad0.98x0.95mm_HandSolder, symbol Device:R
- removed U2: VND9025AJTR, Snapeda:IC_POWERSSO-16_STM-L, symbol Snapeda:VND9025AJTR
- removed U6: JS207011SCQNR, Snapeda:SOIC_SCQNR_CNK, symbol Snapeda:JS207011SCQNR
- added R9: 100k, Resistor_SMD:R_0603_1608Metric_Pad0.98x0.95mm_HandSolder, symbol Device:R
- added S3: JS202011SCQN, Samacsys:JS202011SCQN, symbol Samacsys:JS202011SCQN
- added U6: SISS65DN-T1-GE3, Snapeda:POWERPAK-1212-8S_VIS, symbol Snapeda:SISS65DN-T1-GE3
- U5: footprint Snapeda:RPA0010A-MFG -> Samacsys:TPS56A37RPAR
Connections:
- net +12V power is gone; now on net +12V: D4.1 (K), J3.2
- net +12V pyro sw is gone; now on net +12V pyro: J4.2
- net +12V pyro: no longer J4.1
- net GND: now also S3.1
- net +12V I/O renamed +12V
- net +12V: now also C22.2, C23.2, C24.2, CR1.1, J4.1, U5.11 (VIN), U5.12 (VIN), U5.13 (VIN), U5.8 (VIN), U6.1 (S), U6.2 (S), U6.3 (S)
- removed net +12V main: C22.2, C23.2, C24.2, CR1.1, J3.1, U3.1 (S), U3.2 (S), U3.3 (S), U5.8 (VIN)
- new net: R9.2, U6.4 (G)
- new net: R9.1, S3.2
- new net +VBAT PROTECTED: J3.1, S3.3, U3.1 (S), U3.2 (S), U3.3 (S), U6.5 (D), U6.6 (D), U6.7 (D), U6.8 (D)
- no-connect marks 4 -> 3
Other:
- note removed: "high-side switch"
- moved on the sheet: D4, R16

Commit message: Power rail optimisations
Parts:
- removed R9: 100k, Resistor_SMD:R_0603_1608Metric_Pad0.98x0.95mm_HandSolder, symbol Device:R
- removed U3: SISS65DN-T1-GE3, Snapeda:POWERPAK-1212-8S_VIS, symbol Snapeda:SISS65DN-T1-GE3
- C20: footprint Capacitor_SMD:C_1210_3225Metric_Pad1.33x2.70mm_HandSolder -> Capacitor_SMD:C_0603_1608Metric_Pad1.08x0.95mm_HandSolder
- C21: value 22uF -> 10uF; footprint Capacitor_SMD:C_1210_3225Metric_Pad1.33x2.70mm_HandSolder -> Capacitor_SMD:C_0603_1608Metric_Pad1.08x0.95mm_HandSolder
- L2: footprint Snapeda:IND_SRP1265A-3R3M -> Snapeda:L_Wurth_WE-XHMI-6030
Connections:
- net +12V: now also U6.5 (D), U6.6 (D), U6.7 (D), U6.8 (D); no longer J3.2, U6.1 (S), U6.2 (S), U6.3 (S)
- net +VBAT: now also R8.1, U6.1 (S), U6.2 (S), U6.3 (S)
- net GND: now also J3.2; no longer R8.2
- net gate: now reaches U6.4 (G)
- net gate: now also J3.1, R8.2, S3.2
- removed net +VBAT PROTECTED: J3.1, S3.3, U6.5 (D), U6.6 (D), U6.7 (D), U6.8 (D)
- no-connect marks 3 -> 4
Other:
- note added: "power switch and reverse polarity protection"
- note removed: "power switch"
- note removed: "reverse polarity protection"
- moved on the sheet: C20, C21, R8, S3, U4

Commit message: Final few traces
Parts:
- added R9: 100k, Resistor_SMD:R_0603_1608Metric_Pad0.98x0.95mm_HandSolder, symbol Device:R
- added U11: SISS65DN-T1-GE3, Snapeda:POWERPAK-1212-8S_VIS, symbol Snapeda:SISS65DN-T1-GE3
- D4: value 8.6V -> 8.7V
Connections:
- net +VBAT: now also U11.5 (D), U11.6 (D), U11.7 (D), U11.8 (D); no longer R8.1, U6.1 (S), U6.2 (S), U6.3 (S)
- net GND: now also R9.2
- new net: R9.1, U11.4 (G)
- new net +VBAT safe: R8.1, U11.1 (S), U11.2 (S), U11.3 (S), U6.1 (S), U6.2 (S), U6.3 (S)
Other:
- note added: "Reverse polarity"
- note added: "Switch"
- note removed: "power switch and reverse polarity protection"

Commit message: Final PCB with silkscreen
Connections:
- net +3.3V: now also U4.4 (EPAD)
- net GND: no longer U4.4 (EPAD)
Changed lines of the file:
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@@
-	)
-	(junction
-		(at 19.05 68.58)
-		(diameter 0)
-		(color 0 0 0 0)
 	)
 	(junction
@@
 	(wire
 		(pts
-			(xy 15.24 68.58) (xy 19.05 68.58)
+			(xy 15.24 68.58) (xy 38.1 68.58)
 		)
 		(stroke
@@
 	(wire
 		(pts
-			(xy 19.05 68.58) (xy 19.05 60.96)
-		)
-		(stroke
-			(width 0)
-			(type default)
-		)
-	)
-	(wire
-		(pts
 			(xy 57.15 58.42) (xy 60.96 58.42)
 		)
@@
 		(pts
 			(xy 106.68 101.6) (xy 106.68 111.76)
-		)
-		(stroke
-			(width 0)
-			(type default)
-		)
-	)
-	(wire
-		(pts
-			(xy 38.1 68.58) (xy 19.05 68.58)
 		)
 		(stroke
@@
 					(unit 1)
 				)
+			)
+		)
+	)
+	(symbol
+		(lib_id "power:+3.3V")
+		(at 19.05 60.96 0)
+		(unit 1)
+		(body_style 1)
+		(exclude_from_sim no)
+		(in_bom yes)
+		(on_board yes)
+		(in_pos_files yes)
+		(dnp no)
+		(fields_autoplaced yes)
+		(property "Reference" "#PWR025"
+			(at 19.05 64.77 0)
+			(hide yes)
+			(show_name no)
+			(do_not_autoplace no)
+			(effects
+				(font
+					(size 1.27 1.27)
+				)
+			)
+		)
+		(property "Value" "+3.3V"
+			(at 19.05 55.88 0)
+			(show_name no)
+			(do_not_autoplace no)
+			(effects
+				(font
+					(size 1.27 1.27)
+				)
+			)
+		)
+		(property "Footprint" ""
+			(at 19.05 60.96 0)
+			(hide yes)
+			(show_name no)
+			(do_not_autoplace no)
+			(effects
+				(font
+					(size 1.27 1.27)
+				)
+			)
+		)
+		(property "Datasheet" ""
+			(at 19.05 60.96 0)
+			(hide yes)
+			(show_name no)
+			(do_not_autoplace no)
+			(effects
+				(font
+					(size 1.27 1.27)
+				)
+			)
+		)
+		(property "Description" "Power symbol creates a global label with name \"+3.3V\""
+			(at 19.05 60.96 0)
+			(hide yes)
+			(show_name no)
+			(do_not_autoplace no)
+			(effects
+				(font
+					(size 1.27 1.27)
+				)
+			)
+		)
+		(pin "1"
+		)
+		(instances
+			(project "flight computer"
+				(path "/f20dbb28-4774-4389-9d87-f45a0594cbc0"
+					(reference "#PWR025")
+					(unit 1)
+				)
