File: flight computer/pyros_&_motor.kicad_sch (KiCad schematic)
At the start: 29 parts, among them J10 ED555/2DS, J4 ED555/2DS, J5 ED555/2DS, J6 ED555/2DS, J7 ED555/2DS, J8 ED555/2DS, J9 ED555/2DS, U12 BTM9011EP

Commit message: Finalisation of Schematic
Parts:
- removed C21: 220 uF, Capacitor_SMD:C_0805_2012Metric_Pad1.18x1.45mm_HandSolder, symbol Device:C
- removed J10, J4, J5, J6, J7, J8, J9: ED555/2DS, Snapeda:CONN_ED555&slash_2DS_OST, symbol Snapeda:ED555_2DS
- removed R27, R28, R29, R30: 1k, Resistor_SMD:R_0805_2012Metric_Pad1.20x1.40mm_HandSolder, symbol Device:R
- removed pyro_1, pyro_2, pyro_3, pyro_4: SIA440DJ-T1-GE3, Snapeda:SON_1DJ-T1-GE3_VIS, symbol Snapeda:SIA440DJ-T1-GE3
- added C41: 220uF, Snapeda:CAPMP7343X310N, symbol Snapeda:F931C227MNC
- added F1, F2, F3, F4: Fuse, Fuse:Fuse_1206_3216Metric_Pad1.42x1.75mm_HandSolder, symbol Device:Fuse
- added J11: pyro 1, Samacsys:5452257, symbol Samacsys:5452257
- added J12: pyro 2, Samacsys:5452257, symbol Samacsys:5452257
- added J13: pyro 3, Samacsys:5452257, symbol Samacsys:5452257
- added J14: pyro 4, Samacsys:5452257, symbol Samacsys:5452257
- added J15: motor out, Samacsys:5452257, symbol Samacsys:5452257
- added J16: 5V out, Samacsys:5452257, symbol Samacsys:5452257
- added J17: motor in, Samacsys:5452257, symbol Samacsys:5452257
- added J18: servo 1, Connector_PinHeader_2.54mm:PinHeader_1x03_P2.54mm_Vertical, symbol Connector:Conn_01x03_Pin
- added J19: servo 2, Connector_PinHeader_2.54mm:PinHeader_1x03_P2.54mm_Vertical, symbol Connector:Conn_01x03_Pin
- added J20: servo 3, Connector_PinHeader_2.54mm:PinHeader_1x03_P2.54mm_Vertical, symbol Connector:Conn_01x03_Pin
- added J21: servo 4, Connector_PinHeader_2.54mm:PinHeader_1x03_P2.54mm_Vertical, symbol Connector:Conn_01x03_Pin
- added JP1: SolderJumper_3_Open, Jumper:SolderJumper-3_P1.3mm_Open_Pad1.0x1.5mm, symbol Jumper:SolderJumper_3_Open
- added Q3, Q4, Q5, Q6: SIA440DJ-T1-GE3, Samacsys:SIA440DJT1GE3, symbol Samacsys:SIA440DJ-T1-GE3
- added R35, R36, R37, R38, R45, R46, R47, R48: 1k, Resistor_SMD:R_0805_2012Metric_Pad1.20x1.40mm_HandSolder, symbol Device:R
- R27: renamed from R32; value 50k -> 51k
- R29: renamed from R56; value 50k -> 51k
- R31: renamed from R58; value 50k -> 51k
- R33: renamed from R60; value 50k -> 51k
- renumbered C19 to C38, C20 to C39, C18 to C40, R26 to R22, R31 to R28, R57 to R30, R59 to R32, R61 to R34, U12 to U7
Connections:
- net +5V: now also J16.1, JP1.1 (A)
- net GND: now also C41.2, J16.2, J18.3 (Pin_3), J19.3 (Pin_3), J20.3 (Pin_3), J21.3 (Pin_3), Q3.1 (D_1), Q3.2 (D_2), Q3.5 (D_3), Q3.6 (D_4), Q3.D1 (D_5), Q4.1 (D_1), Q4.2 (D_2), Q4.5 (D_3), Q4.6 (D_4), Q4.D1 (D_5), Q5.1 (D_1), Q5.2 (D_2), Q5.5 (D_3), Q5.6 (D_4), Q5.D1 (D_5), Q6.1 (D_1), Q6.2 (D_2), Q6.5 (D_3), Q6.6 (D_4), Q6.D1 (D_5)
- net motor in a: now also J17.1
- net motor in b: now also J17.2
- net motor out a: now also J15.1
- net motor out b: now also J15.2
- net pyro 1 gate: now also R45.1
- net pyro 2 gate: now also R46.1
- net pyro 3 gate: now also R47.1
- net pyro 4 gate: now also R48.1
- net +12V motor renamed +12V I/O
- net +12V I/O: now also C41.1, JP1.3 (B)
- net pyro 1 source renamed pyro 1 drain
- net pyro 1 drain: now also J11.2, Q3.4 (S_1), Q3.D2 (S_2)
- net pyro 2 source renamed pyro 2 drain
- net pyro 2 drain: now also J12.2, Q4.4 (S_1), Q4.D2 (S_2)
- net pyro 3 source renamed pyro 3 drain
- net pyro 3 drain: now also J13.2, Q5.4 (S_1), Q5.D2 (S_2)
- net pyro 4 source renamed pyro 4 drain
- net pyro 4 drain: now also J14.2, Q6.4 (S_1), Q6.D2 (S_2)
- new net: F4.2, J14.1
- new net: Q6.3 (G), R48.2
- new net: Q3.3 (G), R45.2
- new net: J18.1 (Pin_1), R35.2
- new net: J19.1 (Pin_1), R36.2
- new net: Q4.3 (G), R46.2
- new net: F1.2, J11.1
- new net: F3.2, J13.1
- new net: J21.1 (Pin_1), R38.2
- new net: Q5.3 (G), R47.2
- new net: F2.2, J12.1
- new net: J20.1 (Pin_1), R37.2
- new net +12V pyro sw: F1.1, F2.1, F3.1, F4.1
- new net +5V/+12V: J18.2 (Pin_2), J19.2 (Pin_2), J20.2 (Pin_2), J21.2 (Pin_2), JP1.2 (C)
- new net servo PWM 1: R35.1
- new net servo PWM 2: R36.1
- new net servo PWM 3: R37.1
- new net servo PWM 4: R38.1
Other:
- note added: "pyro headers"
- note added: "servo headers"
- note removed: "headers"
- title: (none) -> pyros & motor
