File: flight computer/sensors_&_communication.kicad_sch (KiCad schematic)
At the start: 34 parts, among them IC3 ADXL375BCCZ-RL, IC4 114993390, J16 SMA-J-P-H-ST-EM1, J17 SMA-J-P-H-ST-EM1, Q7 BSS84, Q8 BSS138, U27 BMP581, U28 74LVC1G07GW_125, U29 MAX-M10S-00B, U30 MAX-M10S-00B, U7 BNO086

Commit message: Finalisation of Schematic
Parts:
- removed C51: 10nF, Capacitor_SMD:C_0805_2012Metric_Pad1.18x1.45mm_HandSolder, symbol Device:C
- removed C52: 47pF, Capacitor_SMD:C_0805_2012Metric_Pad1.18x1.45mm_HandSolder, symbol Device:C
- removed J16: SMA-J-P-H-ST-EM1, Snapeda:SAMTEC_SMA-J-P-H-ST-EM1, symbol Snapeda:SMA-J-P-H-ST-EM1
- removed L5: 27uH, Inductor_SMD:L_0805_2012Metric_Pad1.05x1.20mm_HandSolder, symbol Device:L
- removed Q7: BSS84, Package_TO_SOT_SMD:SOT-23-3, symbol Simulation_SPICE:PMOS
- removed Q8: BSS138, Package_TO_SOT_SMD:SOT-23-3, symbol Simulation_SPICE:NMOS
- removed R53: 10, Resistor_SMD:R_0805_2012Metric_Pad1.20x1.40mm_HandSolder, symbol Device:R
- removed R54: 100k, Resistor_SMD:R_0805_2012Metric_Pad1.20x1.40mm_HandSolder, symbol Device:R
- removed U28: 74LVC1G07GW_125, Snapeda:IC_74LVC1G07GW_125, symbol Snapeda:74LVC1G07GW_125
- removed U29: MAX-M10S-00B, Snapeda:XCVR_MAX-M10S-00B, symbol Snapeda:MAX-M10S-00B
- added C43: 0.1uF, Capacitor_SMD:C_0805_2012Metric_Pad1.18x1.45mm_HandSolder, symbol Device:C
- added CR2: PESD0402-140, Diode_SMD:D_0402_1005Metric_Pad0.77x0.64mm_HandSolder, symbol Snapeda:PESD0402-140
- added CR3: PESD0402-140, Inductor_SMD:L_0402_1005Metric_Pad0.77x0.64mm_HandSolder, symbol Snapeda:PESD0402-140
- added J22: SMA-J-P-H-ST-EM1, Snapeda:SAMTEC_SMA-J-P-H-ST-EM1, symbol Snapeda:SMA-J-P-H-ST-EM1
- added L3: L, Inductor_SMD:L_0402_1005Metric_Pad0.77x0.64mm_HandSolder, symbol Device:L
- added R42: 0, Resistor_SMD:R_0805_2012Metric_Pad1.20x1.40mm_HandSolder, symbol Device:R
- C52: renamed from C53; value 10nF -> 0
- C54: value 10nF -> 0
- IC3: footprint Samacsys:ADXL375BCCZRL -> Snapeda:LGA_CC-14-1_ADI-L
- L4: renamed from L6; value 27uH -> 0; footprint Inductor_SMD:L_0805_2012Metric_Pad1.05x1.20mm_HandSolder -> Inductor_SMD:L_0603_1608Metric_Pad1.05x0.95mm_HandSolder
- R39: renamed from R17; footprint (none) -> Resistor_SMD:R_0805_2012Metric_Pad1.20x1.40mm_HandSolder
- R40: renamed from R18; footprint (none) -> Resistor_SMD:R_0805_2012Metric_Pad1.20x1.40mm_HandSolder
- R41: renamed from R19; footprint (none) -> Resistor_SMD:R_0805_2012Metric_Pad1.20x1.40mm_HandSolder
- U9: renamed from U7; footprint Snapeda:LTST-BILED-15X16 -> Snapeda:IC_BNO086
- renumbered C47 to C42, C55 to C44, C50 to C45, C44 to C46, C61 to C47, C60 to C48, C59 to C49, C58 to C50, C57 to C51, C56 to C53, IC4 to IC2, J17 to J23, R52 to R43, R51 to R44, U30 to U10, U27 to U8
Connections:
- net GND: now also C43.2, CR2.2, CR3.2, J22.2_1, J22.2_2, J22.3_1, J22.3_2
- net at U10.11 (RF_IN): now also CR2.1, J22.1, L3.1
- net at U10.14 (VCC_RF): now also R42.2
- net MAX M10S boot: now reaches U10.18 (~{SAFEBOOT})
- net MAX M10S int: now reaches U10.5 (EXTINT)
- net at C54.1, J23.1, L4.2: now also CR3.1
- net BNO086 INT renamed BNO086 int
- net BNO086 WAKE renamed BNO086 wake
- net MAX M10S RESET renamed MAX M10S reset
- net MAX M10S TIMEPULSE renamed MAX M10S timepulse
- net SX1262 BUSY renamed SX1262 busy
- net SX1262 INT renamed SX1262 int
- net SX1262 RESET renamed SX1262 reset
- net SX1262 RF_SW renamed SX1262 rf switch
- new net: C43.1, L3.2, R42.1
- no-connect marks 18 -> 12
Other:
- note added: "GNSS"
- title: (none) -> sensors & communication
- moved on the sheet: C44, C45, J23, U10
