File: flight computer/flight computer.kicad_pcb (KiCad board)
At the start: 4 copper layers, 43.2 x 99.1 mm, 170 parts, among them IC1 AT25SF128A-SHB-T, IC2 114993390, IC3 ADXL375BCCZ-RL, J1 JST, J10 Micro_SD_Card, J11 pyro 1, J12 pyro 2, J13 pyro 3, J14 pyro 4, J15 motor out, J16 5V out, J17 motor in, J18 servo 1, J19 servo 2, J2 battery in, J20 servo 3, J21 servo 4, J22 SMA-J-P-H-ST-EM1, J23 SMA-J-P-H-ST-EM1, J3 battery sw, J4 pyro sw, J5 12V out, J6 5V out, J7 3.3V out, J8 USB_C_Receptacle_USB2.0_16P, J9 GPIO, Q1 NMOS, Q2 PMOS, Q3 SIA440DJ-T1-GE3, Q4 SIA440DJ-T1-GE3, Q5 SIA440DJ-T1-GE3, Q6 SIA440DJ-T1-GE3, U1 RP2350B, U10 MAX-M10S-00B, U2 VND9025AJTR, U3 SISS65DN-T1-GE3, U4 AZ1117CH-3.3TRG1, U5 TPS56A37RPAR, U6 JS207011SCQNR, U7 BTM9011EP, U8 BMP581, U9 BNO086, Y1 ABM8G-12.000MHZ-18-D2Y-T

Commit message: General progress on the PCB
Parts:
- removed D2, D3: D_Schottky, Diode_SMD:D_SOD-123
- removed Q1: NMOS, Package_TO_SOT_SMD:SOT-23-3
- removed R11: 200k, Resistor_SMD:R_0805_2012Metric_Pad1.20x1.40mm_HandSolder
- removed R9: 330, Resistor_SMD:R_0805_2012Metric_Pad1.20x1.40mm_HandSolder
- added R24: 0, Resistor_SMD:R_0603_1608Metric_Pad0.98x0.95mm_HandSolder, B.Cu at (215.7, 89.4)
- added R25: 0, Resistor_SMD:R_0603_1608Metric_Pad0.98x0.95mm_HandSolder, B.Cu at (205.2, 88.6)
- C1, C10, C11, C12, C13, C14, C15, C16, C17, C18, C19, C2, C24, C25, C26, C27, C28, C29, C3, C32, C33, C34, C35, C36, C37, C38, C39, C4, C40, C42, C43, C44, C45, C46, C47, C48, C49, C5, C50, C51, C52, C53, C54, C6, C7, C8, C9: footprint Capacitor_SMD:C_0805_2012Metric_Pad1.18x1.45mm_HandSolder -> Capacitor_SMD:C_0603_1608Metric_Pad1.08x0.95mm_HandSolder
- C20, C22, C23: footprint Capacitor_SMD:C_1206_3216Metric_Pad1.33x1.80mm_HandSolder -> Capacitor_SMD:C_1210_3225Metric_Pad1.33x2.70mm_HandSolder
- R1, R10, R12, R13, R14, R15, R16, R17, R18, R19, R2, R20, R21, R22, R23, R27, R28, R29, R3, R30, R31, R32, R33, R34, R35, R36, R37, R38, R39, R40, R41, R42, R43, R44, R45, R46, R47, R48, R6, R7, R8: footprint Resistor_SMD:R_0805_2012Metric_Pad1.20x1.40mm_HandSolder -> Resistor_SMD:R_0603_1608Metric_Pad0.98x0.95mm_HandSolder
- R4, R5: footprint Resistor_SMD:R_0805_2012Metric_Pad1.20x1.40mm_HandSolder -> Resistor_SMD:R_0603_1608Metric_Pad0.98x0.95mm_HandSolder; moved to F.Cu
- moved Q2 125.1 mm to (217.9, 82.5), turned to 90 degrees
- moved R38 114.0 mm to (210.4, 126.6), turned to 90 degrees
- moved D5 113.4 mm to (202.2, 123.8)
- moved R37 109.2 mm to (204.1, 126.6), turned to 90 degrees
- moved R21 105.1 mm to (218.1, 102.0), turned to -90 degrees
- moved R20 105.1 mm to (218.1, 98.7), turned to 90 degrees
- moved R1 101.9 mm to (215.4, 110.5)
- moved R36 100.1 mm to (192.7, 126.6), turned to 90 degrees
- moved D1 95.8 mm to (188.5, 67.3), turned to -90 degrees
- moved R19 95.0 mm to (199.7, 128.9), turned to -90 degrees
- moved R18 94.0 mm to (197.1, 128.9), turned to -90 degrees
- moved R35 81.9 mm to (186.3, 126.6), turned to 90 degrees
- moved R7 77.6 mm to (190.5, 68.1), turned to 90 degrees
- moved R2 74.9 mm to (188.2, 109.5), turned to 90 degrees
- moved IC1 73.4 mm to (262.9, 111.3), turned to 0 degrees
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Connections:
- net /USB_DM renamed /USB_DN
- C27 pad 2: Net-(D3-A) -> Net-(Q2-G)
- C28 pad 2: Net-(U5-BOOT) -> Net-(C28-Pad2)
- Q2 pad 2: Net-(D3-A) -> Net-(Q2-G)
- R12 pad 2: Net-(D3-A) -> Net-(Q2-G)
- R13 pad 1: Net-(C29-Pad2) -> Net-(R13-Pad1)
- R14 pad 2: Net-(C29-Pad2) -> Net-(R13-Pad1)
- U1 pad 40: /pin out 1 -> /pin out 2
- U1 pad 42: /pin out 2 -> /pin out 1
- U2 pad 10: +12V I/O -> +12V pyro
- U2 pad 11: +12V I/O -> +12V pyro
- U2 pad 12: +12V I/O -> +12V pyro
- U2 pad 13: +12V pyro -> +12V I/O
- U2 pad 14: +12V pyro -> +12V I/O
- U2 pad 15: +12V pyro -> +12V I/O
- U2 pad 16: +12V pyro -> +12V I/O
- U2 pad 9: +12V I/O -> +12V pyro
- U6 pad 1: Net-(D2-K) -> Net-(Q2-G)
- U6 pad 5: Net-(D2-K) -> Net-(Q2-G)
Routing:
- net +12V power: track 0.00 -> 55.4 mm, vias 0 -> 1
- net Net-(Q2-G): track 0.00 -> 39.4 mm, vias 0 -> 3
- net GND: track 0.00 -> 29.2 mm, vias 0 -> 163
- net /pin out 1: track 0.00 -> 21.1 mm, vias 0 -> 1
- net /pin out 2: track 0.00 -> 20.2 mm, vias 0 -> 1
- net +5V: track 0.00 -> 19.1 mm, vias 0 -> 12
- net Net-(S2-NO_1): track 0.00 -> 18.4 mm
- net Net-(S2-COM_1): track 0.00 -> 10.6 mm, vias 0 -> 1
- net Net-(D1-A): track 0.00 -> 7.58 mm
- net /power signal: track 0.00 -> 7.37 mm, vias 0 -> 1
- net Net-(U5-SW): track 0.00 -> 7.29 mm
- net Net-(LED1-DOUT): track 0.00 -> 6.56 mm
- net Net-(LED2-DOUT): track 0.00 -> 6.56 mm
- net Net-(U5-SS): track 0.00 -> 5.68 mm
- net Net-(U5-PG): track 0.00 -> 5.46 mm
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- added copper zone on B.Cu, net +12V I/O
- added copper zone on F.Cu, net +12V I/O
- added copper zone on B.Cu, net +12V main
- added copper zone on B.Cu, net +12V pyro
- added copper zone on F.Cu, net +12V pyro sw
- added copper zone on B.Cu, net +3.3V
- added copper zone on In1.Cu, net +3.3V
- added copper zone on B.Cu, net +5V
- added copper zone on F.Cu, net +5V
- added copper zone on In1.Cu, net +5V
- added copper zone on In2.Cu, net +5V
- added copper zone on F.Cu, net +5V/+12V
- added copper zone on B.Cu, net +VBAT
- added copper zone on B.Cu, net /motor out a
- added copper zone on B.Cu, net /motor out b
- added copper zone on B.Cu, net GND
- added copper zone on F.Cu, net GND
- added copper zone on In1.Cu, net GND
- added copper zone on In2.Cu, net GND
- added copper zone on B.Cu, net Net-(C28-Pad2)
- added copper zone on In1.Cu, net Net-(D5-A)
- added copper zone on B.Cu, net Net-(U5-BOOT)
- added copper zone on B.Cu, net Net-(U5-SW)

Commit message: Tried a more effective layout
Parts:
- removed C26, C27, C32, C33, C34, C35: 0.1uF, Capacitor_SMD:C_0603_1608Metric_Pad1.08x0.95mm_HandSolder
- removed D1: D_Schottky, Diode_SMD:D_SOD-123
- removed Q2: PMOS, Package_TO_SOT_SMD:SOT-23-3
- removed R12: 100k, Resistor_SMD:R_0603_1608Metric_Pad0.98x0.95mm_HandSolder
- removed R7: 4.7k, Resistor_SMD:R_0603_1608Metric_Pad0.98x0.95mm_HandSolder
- removed U2: VND9025AJTR, Snapeda:IC_POWERSSO-16_STM-L
- added G***: LOGO, LOGO, F.Cu at (198.4, 58.9)
- added R9: 100k, Resistor_SMD:R_0603_1608Metric_Pad0.98x0.95mm_HandSolder, B.Cu at (180.9, 57.4)
- added S3: JS202011SCQN, Samacsys:JS202011SCQN, F.Cu at (198.4, 105.4)
- C1, C10, C11, C12, C13, C14, C15, C18, C19, C3, C36, C37, C4, C43, C5, C52, C54, C6, C7, C8, C9, CR2, CR3, L3, L4, R17, R3, R42: moved to F.Cu
- F1, F2, F3, F4, R4, R5: moved to B.Cu
- U1: footprint Package_DFN_QFN:QFN-80-1EP_10x10mm_P0.4mm_EP3.4x3.4mm -> Package_DFN_QFN:QFN-80-1EP_10x10mm_P0.4mm_EP3.4x3.4mm_ThermalVias
- U5: footprint Snapeda:RPA0010A-MFG -> Samacsys:TPS56A37RPAR
- U6: value JS207011SCQNR -> SISS65DN-T1-GE3; footprint Snapeda:SOIC_SCQNR_CNK -> Snapeda:POWERPAK-1212-8S_VIS; moved to B.Cu
- moved R27 122.1 mm to (215.9, 47.8), turned to 0 degrees
- moved R45 119.6 mm to (208.4, 54.9)
- moved R46 119.4 mm to (208.4, 58.9)
- moved R28 119.3 mm to (215.9, 46.3)
- moved R47 119.1 mm to (208.4, 62.9)
- moved R48 118.9 mm to (208.4, 66.9)
- moved R30 118.1 mm to (215.9, 56.4)
- moved C53 117.8 mm to (205.4, 72.9), turned to -90 degrees
- moved R32 117.0 mm to (215.9, 66.7)
- moved R29 116.9 mm to (215.9, 57.9), turned to 0 degrees
- moved C51 116.4 mm to (203.9, 72.9), turned to -90 degrees
- moved R34 116.0 mm to (215.9, 76.8)
- moved R31 116.0 mm to (215.9, 68.2), turned to 0 degrees
- moved C8 115.9 mm to (113.0, 176.9), turned to 0 degrees
- moved C9 115.4 mm to (113.0, 179.4), turned to 0 degrees
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Connections:
- net Net-(U1-USB_DN) renamed /MCU_DN
- net Net-(U1-USB_DP) renamed /MCU_DP
- C22 pad 2: +12V main -> +12V
- C23 pad 2: +12V main -> +12V
- C24 pad 2: +12V main -> +12V
- C38 pad 1: +12V I/O -> +12V
- C39 pad 1: +12V I/O -> +12V
- C41 pad 1: +12V I/O -> +12V
- CR1 pad 1: +12V main -> +12V
- D4 pad 1: +12V power -> +12V
- F1 pad 1: +12V pyro sw -> +12V pyro
- F2 pad 1: +12V pyro sw -> +12V pyro
- F3 pad 1: +12V pyro sw -> +12V pyro
- F4 pad 1: +12V pyro sw -> +12V pyro
- J3 pad 1: +12V main -> +VBAT PROTECTED
- J3 pad 2: +12V power -> +12V
- J4 pad 1: +12V pyro -> +12V
- J4 pad 2: +12V pyro sw -> +12V pyro
- J5 pad 1: +12V I/O -> +12V
- JP1 pad 1: +5V -> +12V
- JP1 pad 3: +12V I/O -> +5V
- R1 pad 1: Net-(S2-COM_1) -> Net-(S2-COM_2)
- R2 pad 2: Net-(S1-NO_1) -> Net-(S1-NO_2)
- S1 pad 1: Net-(S1-NO_1) -> unconnected-(S1-NO_1-Pad1)
- S1 pad 2: Net-(S1-NO_1) -> Net-(S1-NO_2)
- S1 pad 4: GND -> unconnected-(S1-COM_2-Pad4)
- S2 pad 2: Net-(S2-NO_1) -> unconnected-(S2-NO_2-Pad2)
- S2 pad 3: Net-(S2-COM_1) -> unconnected-(S2-COM_1-Pad3)
- S2 pad 4: Net-(S2-COM_1) -> Net-(S2-COM_2)
- U1 pad 1: /MAX M10S TX -> /motor in a
- U1 pad 11: /servo PWM 1 -> unconnected-(U1-GPIO12-Pad11)
- U1 pad 12: /servo PWM 2 -> unconnected-(U1-GPIO13-Pad12)
- U1 pad 13: /pyro 1 gate -> unconnected-(U1-GPIO14-Pad13)
- U1 pad 14: /pyro 2 gate -> unconnected-(U1-GPIO15-Pad14)
- U1 pad 16: /pyro 3 gate -> unconnected-(U1-GPIO16-Pad16)
- U1 pad 17: /pyro 4 gate -> unconnected-(U1-GPIO17-Pad17)
- U1 pad 18: /servo PWM 3 -> unconnected-(U1-GPIO18-Pad18)
- U1 pad 19: /servo PWM 4 -> unconnected-(U1-GPIO19-Pad19)
- U1 pad 2: /MAX M10S RX -> /motor in b
- U1 pad 20: /VND9025 IN0 -> unconnected-(U1-GPIO20-Pad20)
- U1 pad 21: /VND9025 fault -> unconnected-(U1-GPIO21-Pad21)
- U1 pad 22: /VND9025 IN1 -> unconnected-(U1-GPIO22-Pad22)
- U1 pad 23: /SX1262 rf switch -> unconnected-(U1-GPIO23-Pad23)
- U1 pad 25: /SX1262 reset -> unconnected-(U1-GPIO24-Pad25)
- U1 pad 26: /SX1262 CS -> unconnected-(U1-GPIO25-Pad26)
- U1 pad 27: /SX1262 busy -> unconnected-(U1-GPIO26-Pad27)
- U1 pad 28: /SX1262 int -> unconnected-(U1-GPIO27-Pad28)
- U1 pad 3: /MAX M10S timepulse -> /pin out 2
- U1 pad 36: /BNO086 wake -> /SCK
- U1 pad 37: /BNO086 int -> /MISO
- U1 pad 39: /ADXL375 CS -> /MOSI
- U1 pad 4: /MAX M10S int -> /pin out 1
- U1 pad 40: /pin out 2 -> /BNO086 int
- U1 pad 42: /pin out 1 -> /BNO086 wake
- U1 pad 43: /SD CLK -> /SD DAT1
- U1 pad 44: /SD CMD -> /SD DAT0
- U1 pad 45: /SD DAT0 -> /SD CLK
- U1 pad 46: /SD DAT1 -> /SD CMD
- U1 pad 47: /SD DAT2 -> /SD DAT3
- U1 pad 48: /SD DAT3 -> /SD DAT2
- U1 pad 55: /BTM9011EP CS -> unconnected-(U1-GPIO44/ADC4-Pad55)
- U1 pad 56: /BTM9011EP IS -> unconnected-(U1-GPIO45/ADC5-Pad56)
- U1 pad 57: /power signal -> /BTM9011EP CS
- U1 pad 58: /power controller -> /BTM9011EP IS
- U1 pad 6: /MAX M10S reset -> unconnected-(U1-GPIO8-Pad6)
- U1 pad 7: /MAX M10S boot -> unconnected-(U1-GPIO9-Pad7)
- U1 pad 77: /MISO -> /servo PWM 1
- U1 pad 78: /MOSI -> /servo PWM 2
- U1 pad 79: /SCK -> /servo PWM 3
- U1 pad 8: /motor in a -> unconnected-(U1-GPIO10-Pad8)
- U1 pad 80: /BMP581 CS -> /servo PWM 4
- U1 pad 9: /motor in b -> unconnected-(U1-GPIO11-Pad9)
- U3 pad 1: +12V main -> +VBAT PROTECTED
- U3 pad 2: +12V main -> +VBAT PROTECTED
- U3 pad 3: +12V main -> +VBAT PROTECTED
- U5 pad 8: +12V main -> +12V
- U6 pad 1: Net-(Q2-G) -> +12V
- U6 pad 2: GND -> +12V
- U6 pad 3: GND -> +12V
- U6 pad 4: GND -> Net-(U6-G)
- U6 pad 5: Net-(Q2-G) -> +VBAT PROTECTED
- U6 pad 6: GND -> +VBAT PROTECTED
- U6 pad 7: GND -> +VBAT PROTECTED
- U6 pad 8: GND -> +VBAT PROTECTED
- U7 pad 11: +12V I/O -> +12V
- U7 pad 12: +12V I/O -> +12V
Routing:
- net +VBAT PROTECTED: track 0.00 -> 61.7 mm, vias 0 -> 1
- net Net-(R9-Pad1): track 0.00 -> 55.6 mm, vias 0 -> 2
- net /MISO: track 1.25 -> 56.6 mm, vias 1 -> 4
- net +12V power: track 55.4 -> 0.00 mm, vias 1 -> 0
- net /SCK: track 1.49 -> 53.2 mm, vias 1 -> 2
- net /MOSI: track 1.68 -> 51.2 mm, vias 1 -> 3
- net Net-(Q2-G): track 39.4 -> 0.00 mm, vias 3 -> 0
- net /motor in b: track 0.00 -> 36.9 mm, vias 0 -> 1
- net /MCU_DN: track 0.00 -> 34.5 mm, vias 0 -> 1
- net /MCU_DP: track 0.00 -> 34.4 mm, vias 0 -> 1
- net /motor in a: track 0.00 -> 31.2 mm, vias 0 -> 1
- net /servo PWM 1: track 0.85 -> 31.8 mm
- net /servo PWM 2: track 0.85 -> 31.3 mm
- net /servo PWM 4: track 0.86 -> 30.4 mm
- net /servo PWM 3: track 0.85 -> 30.2 mm
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- added copper zone on B.Cu, net +12V
- added copper zone on F.Cu, net +12V
- added copper zone on In2.Cu, net +12V pyro
- added copper zone on B.Cu, net +VBAT PROTECTED
- added copper zone on F.Cu, net /pyro 1 drain
- added copper zone on F.Cu, net /pyro 2 drain
- added copper zone on F.Cu, net /pyro 3 drain
- added copper zone on F.Cu, net /pyro 4 drain
- added copper zone on B.Cu, net Net-(D5-A)
- added copper zone on F.Cu, net Net-(D5-A)
- removed copper zone on B.Cu, net +12V I/O
- removed copper zone on F.Cu, net +12V I/O
- removed copper zone on B.Cu, net +12V main
- removed copper zone on F.Cu, net +12V pyro sw
- removed copper zone on In1.Cu, net +3.3V
- removed copper zone on In1.Cu, net +5V
- removed copper zone on In2.Cu, net +5V
- removed copper zone on B.Cu, net Net-(C28-Pad2)
- removed copper zone on In1.Cu, net Net-(D5-A)
- removed copper zone on B.Cu, net Net-(U5-BOOT)

Commit message: Power rail optimisations
Parts:
- removed G***: LOGO, LOGO
- removed JP1: SolderJumper_3_Open, Jumper:SolderJumper-3_P1.3mm_Open_Pad1.0x1.5mm
- removed R1, R2, R20, R21: 1k, Resistor_SMD:R_0603_1608Metric_Pad0.98x0.95mm_HandSolder
- removed R9: 100k, Resistor_SMD:R_0603_1608Metric_Pad0.98x0.95mm_HandSolder
- removed U3: SISS65DN-T1-GE3, Snapeda:POWERPAK-1212-8S_VIS
- added R11: 1k, Resistor_SMD:R_0603_1608Metric_Pad0.98x0.95mm_HandSolder, B.Cu at (256.2, 113.8)
- added R7: 1k, Resistor_SMD:R_0603_1608Metric_Pad0.98x0.95mm_HandSolder, B.Cu at (254.4, 112.0)
- C1, C10, C11, C12, C13, C14, C15, C18, C19, C3, C36, C37, C4, C5, C6, C7, C8, C9, R17, R3: moved to B.Cu
- C20: footprint Capacitor_SMD:C_1210_3225Metric_Pad1.33x2.70mm_HandSolder -> Capacitor_SMD:C_0603_1608Metric_Pad1.08x0.95mm_HandSolder
- C21: value 22uF -> 10uF; footprint Capacitor_SMD:C_1210_3225Metric_Pad1.33x2.70mm_HandSolder -> Capacitor_SMD:C_0603_1608Metric_Pad1.08x0.95mm_HandSolder
- C40, R22, R45, R46, R47, R48: moved to F.Cu
- L2: footprint Snapeda:IND_SRP1265A-3R3M -> Snapeda:L_Wurth_WE-XHMI-6030
- U1: footprint Package_DFN_QFN:QFN-80-1EP_10x10mm_P0.4mm_EP3.4x3.4mm_ThermalVias -> Package_DFN_QFN:QFN-80-1EP_10x10mm_P0.4mm_EP3.4x3.4mm
- Y1: value ABM8G-12.000MHZ-18-D2Y-T -> ABM8-272-T3; footprint Snapeda:CRYSTAL_ABM8G_ABR-L -> Samacsys:ABM8272T3
- moved C19 235.9 mm to (261.1, 112.5), turned to -135 degrees
- moved C18 234.3 mm to (259.3, 110.7), turned to -135 degrees
- moved C14 158.1 mm to (267.7, 112.9), turned to -135 degrees
- moved C36 153.1 mm to (184.9, 79.9), turned to 90 degrees
- moved C37 151.3 mm to (183.4, 79.9), turned to 90 degrees
- moved R17 149.4 mm to (191.9, 66.9), turned to -90 degrees
- moved C10 134.8 mm to (203.5, 82.0), turned to 45 degrees
- moved C8 131.1 mm to (205.6, 84.1), turned to 45 degrees
- moved C5 125.8 mm to (204.5, 83.0), turned to 45 degrees
- moved C7 125.2 mm to (208.4, 93.2), turned to -45 degrees
- moved C12 120.6 mm to (195.1, 98.5), turned to -135 degrees
- moved C11 120.0 mm to (188.9, 91.5), turned to -135 degrees
- moved C15 117.4 mm to (198.4, 79.5), turned to 45 degrees
- moved C9 115.5 mm to (191.3, 94.5), turned to -135 degrees
- moved C3 112.3 mm to (191.3, 83.8), turned to 135 degrees
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Connections:
- J10 pad SH: GND -> unconnected-(J10-SHIELD-PadSH)_3
- J18 pad 2: +5V/+12V -> +5V
- J19 pad 2: +5V/+12V -> +5V
- J20 pad 2: +5V/+12V -> +5V
- J21 pad 2: +5V/+12V -> +5V
- J3 pad 1: +VBAT PROTECTED -> /gate
- J3 pad 2: +12V -> GND
- J9 pad 1: Net-(J9-Pad1) -> /pin out 1
- J9 pad 2: Net-(J9-Pad2) -> /pin out 2
- R8 pad 1: Net-(U3-G) -> +VBAT
- R8 pad 2: GND -> /gate
- S1 pad 2: Net-(S1-NO_2) -> /QSPI_SS
- S1 pad 3: GND -> Net-(S1-COM_1)
- S2 pad 4: Net-(S2-COM_2) -> GND
- S3 pad 2: Net-(R9-Pad1) -> /gate
- S3 pad 3: +VBAT PROTECTED -> unconnected-(S3-Pad3)
- U1 pad 1: /motor in a -> unconnected-(U1-GPIO4-Pad1)
- U1 pad 2: /motor in b -> unconnected-(U1-GPIO5-Pad2)
- U1 pad 3: /pin out 2 -> unconnected-(U1-GPIO6-Pad3)
- U1 pad 35: Net-(S2-NO_1) -> Net-(U1-RUN)
- U1 pad 36: /SCK -> unconnected-(U1-GPIO28-Pad36)
- U1 pad 37: /MISO -> unconnected-(U1-GPIO29-Pad37)
- U1 pad 38: /BNO086 CS -> unconnected-(U1-GPIO30-Pad38)
- U1 pad 39: /MOSI -> unconnected-(U1-GPIO31-Pad39)
- U1 pad 4: /pin out 1 -> unconnected-(U1-GPIO7-Pad4)
- U1 pad 40: /BNO086 int -> unconnected-(U1-GPIO32-Pad40)
- U1 pad 42: /BNO086 wake -> unconnected-(U1-GPIO33-Pad42)
- U1 pad 43: /SD DAT1 -> unconnected-(U1-GPIO34-Pad43)
- U1 pad 44: /SD DAT0 -> unconnected-(U1-GPIO35-Pad44)
- U1 pad 45: /SD CLK -> unconnected-(U1-GPIO36-Pad45)
- U1 pad 46: /SD CMD -> unconnected-(U1-GPIO37-Pad46)
- U1 pad 47: /SD DAT3 -> unconnected-(U1-GPIO38-Pad47)
- U1 pad 48: /SD DAT2 -> unconnected-(U1-GPIO39-Pad48)
- U1 pad 49: /pyro 1 continuity -> unconnected-(U1-GPIO40/ADC0-Pad49)
- U1 pad 52: /pyro 2 continuity -> unconnected-(U1-GPIO41/ADC1-Pad52)
- U1 pad 53: /pyro 3 continuity -> unconnected-(U1-GPIO42/ADC2-Pad53)
- U1 pad 54: /pyro 4 continuity -> unconnected-(U1-GPIO43/ADC3-Pad54)
- U1 pad 57: /BTM9011EP CS -> unconnected-(U1-GPIO46/ADC6-Pad57)
- U1 pad 58: /BTM9011EP IS -> unconnected-(U1-GPIO47/ADC7-Pad58)
- U1 pad 77: /servo PWM 1 -> unconnected-(U1-GPIO0-Pad77)
- U1 pad 78: /servo PWM 2 -> unconnected-(U1-GPIO1-Pad78)
- U1 pad 79: /servo PWM 3 -> unconnected-(U1-GPIO2-Pad79)
- U1 pad 80: /servo PWM 4 -> unconnected-(U1-GPIO3-Pad80)
- U6 pad 1: +12V -> +VBAT
- U6 pad 2: +12V -> +VBAT
- U6 pad 3: +12V -> +VBAT
- U6 pad 4: Net-(U6-G) -> /gate
- U6 pad 5: +VBAT PROTECTED -> +12V
- U6 pad 6: +VBAT PROTECTED -> +12V
- U6 pad 7: +VBAT PROTECTED -> +12V
- U6 pad 8: +VBAT PROTECTED -> +12V
Routing:
- net +VBAT PROTECTED: track 61.7 -> 0.00 mm, vias 1 -> 0
- net Net-(R9-Pad1): track 55.6 -> 0.00 mm, vias 2 -> 0
- net /MISO: track 56.6 -> 1.17 mm, vias 4 -> 1
- net /SCK: track 53.2 -> 0.00 mm, vias 2 -> 0
- net /MOSI: track 51.2 -> 0.00 mm, vias 3 -> 0
- net /motor in b: track 36.9 -> 0.00 mm, vias 1 -> 0
- net /MCU_DN: track 34.5 -> 0.00 mm, vias 1 -> 0
- net /MCU_DP: track 34.4 -> 0.00 mm, vias 1 -> 0
- net GND: track 44.5 -> 11.8 mm, vias 136 -> 114
- net /motor in a: track 31.2 -> 0.00 mm, vias 1 -> 0
- net /servo PWM 1: track 31.8 -> 1.09 mm
- net /servo PWM 2: track 31.3 -> 1.09 mm
- net /servo PWM 4: track 30.4 -> 1.09 mm
- net /servo PWM 3: track 30.2 -> 1.09 mm
- net /SWDIO: track 27.3 -> 0.00 mm
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- added copper zone on F.Cu, net +1.1V
- added copper zone on F.Cu, net +3.3V
- removed copper zone on F.Cu, net +12V
- removed copper zone on F.Cu, net +5V
- removed copper zone on F.Cu, net +5V/+12V
- removed copper zone on B.Cu, net +VBAT PROTECTED
