File: flight computer/flight computer.kicad_pcb (KiCad board)
At the start: 4 copper layers, 43.2 x 99.1 mm, 153 parts, among them IC1 AT25SF128A-SHB-T, IC2 114993390, IC3 ADXL375BCCZ-RL, J1 JST, J10 Micro_SD_Card, J11 pyro 1, J12 pyro 2, J13 pyro 3, J14 pyro 4, J15 motor out, J16 5V out, J17 motor in, J18 servo 1, J19 servo 2, J2 battery in, J20 servo 3, J21 servo 4, J22 SMA-J-P-H-ST-EM1, J23 SMA-J-P-H-ST-EM1, J3 battery sw, J4 pyro sw, J5 12V out, J6 5V out, J7 3.3V out, J8 USB_C_Receptacle_USB2.0_16P, J9 GPIO, Q3 SIA440DJ-T1-GE3, Q4 SIA440DJ-T1-GE3, Q5 SIA440DJ-T1-GE3, Q6 SIA440DJ-T1-GE3, U1 RP2350B, U10 MAX-M10S-00B, U4 AZ1117CH-3.3TRG1, U5 TPS56A37RPAR, U6 SISS65DN-T1-GE3, U7 BTM9011EP, U8 BMP581, U9 BNO086, Y1 ABM8-272-T3

Commit message: Designed RF segment
Parts:
- removed CR2: PESD0402-140, Diode_SMD:D_0402_1005Metric_Pad0.77x0.64mm_HandSolder
- added D2: D_TVS, Diode_SMD:D_0603_1608Metric_Pad1.05x0.95mm_HandSolder, B.Cu at (205.3, 39.5)
- L3: footprint Inductor_SMD:L_0402_1005Metric_Pad0.77x0.64mm_HandSolder -> Inductor_SMD:L_0603_1608Metric_Pad1.05x0.95mm_HandSolder
- moved R42 43.6 mm to (209.2, 40.4), turned to -90 degrees
- moved C43 42.9 mm to (207.7, 40.4), turned to 90 degrees
- moved L3 38.3 mm to (205.3, 41.3), turned to 0 degrees
- moved R17 27.0 mm to (191.9, 66.7)
- moved U10 16.8 mm to (207.7, 48.4), turned to 90 degrees
- moved IC2 12.9 mm to (193.0, 48.9), turned to 180 degrees
- moved C52 11.1 mm to (194.8, 41.3)
- moved C54 11.1 mm to (194.8, 39.5)
- moved L4 11.0 mm to (192.4, 40.4)
- moved J22 11.0 mm to (204.4, 36.2)
- moved J23 11.0 mm to (192.4, 36.2)
- moved D1 11.0 mm to (190.9, 40.4)
- moved LS1 1.12 mm to (199.4, 62.4), turned to -90 degrees
- moved R8 0.71 mm to (182.9, 57.4)
- moved U6 0.71 mm to (185.9, 57.4)
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Connections:
- U1 pad 11: /SX1262 int -> /MAX M10S boot
- U1 pad 12: unconnected-(U1-GPIO13-Pad12) -> /MAX M10S reset
- U1 pad 13: /SCK -> unconnected-(U1-GPIO14-Pad13)
- U1 pad 14: /ADXL375 CS -> unconnected-(U1-GPIO15-Pad14)
- U1 pad 16: /BMP581 CS -> unconnected-(U1-GPIO16-Pad16)
- U1 pad 17: /BNO086 CS -> unconnected-(U1-GPIO17-Pad17)
- U1 pad 18: /MOSI -> unconnected-(U1-GPIO18-Pad18)
- U1 pad 19: /MISO -> unconnected-(U1-GPIO19-Pad19)
- U1 pad 20: /BNO086 int -> unconnected-(U1-GPIO20-Pad20)
- U1 pad 21: /BNO086 wake -> /BNO086 int
- U1 pad 22: /MAX M10S boot -> /BNO086 wake
- U1 pad 23: /MAX M10S TX -> /SX1262 CS
- U1 pad 25: /MAX M10S RX -> /SX1262 reset
- U1 pad 26: /MAX M10S timepulse -> /SX1262 rf switch
- U1 pad 27: /MAX M10S int -> /SX1262 int
- U1 pad 28: /MAX M10S reset -> /SX1262 busy
- U1 pad 6: /SX1262 rf switch -> /MAX M10S int
- U1 pad 7: /SX1262 reset -> /MAX M10S timepulse
- U1 pad 8: /SX1262 CS -> /MAX M10S RX
- U1 pad 9: /SX1262 busy -> /MAX M10S TX
Routing:
- net /MOSI: track 84.1 -> 14.1 mm, vias 4 -> 2
- net /MISO: track 81.0 -> 14.9 mm, vias 5 -> 3
- net /SCK: track 94.9 -> 36.9 mm, vias 3 -> 2
- net /SX1262 int: track 39.8 -> 54.6 mm
- net /BNO086 CS: track 14.5 -> 0.00 mm
- net /SX1262 busy: track 41.1 -> 54.8 mm
- net /MAX M10S boot: track 34.3 -> 47.2 mm
- net /BMP581 CS: track 12.2 -> 0.00 mm, vias 2 -> 0
- net /ADXL375 CS: track 12.2 -> 0.00 mm, vias 2 -> 0
- net /MAX M10S reset: track 46.5 -> 37.3 mm
- net Net-(IC2-ANT): track 12.2 -> 3.66 mm
- net Net-(D2-A2): track 0.00 -> 7.96 mm
- net /SX1262 rf switch: track 45.7 -> 52.7 mm
- net Net-(LED2-DOUT): track 0.00 -> 6.51 mm
- net Net-(LED1-DOUT): track 0.12 -> 6.51 mm
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- added copper zone on In2.Cu, net +1.1V
- removed copper zone on In1.Cu, net +1.1V

Commit message: Final few traces
Parts:
- removed Q3: SIA440DJ-T1-GE3, Samacsys:SIA440DJT1GE3
- removed R45: 1k, Resistor_SMD:R_0603_1608Metric_Pad0.98x0.95mm_HandSolder
- added Q7: SIA440DJ-T1-GE3, Samacsys:SIA440DJT1GE3, F.Cu at (206.4, 52.6)
- added R12: 10k, Resistor_SMD:R_0603_1608Metric_Pad0.98x0.95mm_HandSolder, B.Cu at (208.8, 84.9)
- added R49: 1k, Resistor_SMD:R_0603_1608Metric_Pad0.98x0.95mm_HandSolder, B.Cu at (207.7, 83.8)
- added R50: 100k, Resistor_SMD:R_0603_1608Metric_Pad0.98x0.95mm_HandSolder, B.Cu at (208.9, 70.9)
- added R51: 100k, Resistor_SMD:R_0603_1608Metric_Pad0.98x0.95mm_HandSolder, B.Cu at (207.4, 70.9)
- added R52: 100k, Resistor_SMD:R_0603_1608Metric_Pad0.98x0.95mm_HandSolder, B.Cu at (205.9, 70.9)
- added R53: 100k, Resistor_SMD:R_0603_1608Metric_Pad0.98x0.95mm_HandSolder, B.Cu at (210.4, 70.9)
- added R9: 100k, Resistor_SMD:R_0603_1608Metric_Pad0.98x0.95mm_HandSolder, B.Cu at (180.4, 46.4)
- added U11: SISS65DN-T1-GE3, Snapeda:POWERPAK-1212-8S_VIS, B.Cu at (184.4, 47.0)
- C16, C17: value 27pF -> 15pF
- C43: value 0.1uF -> 10nF
- D4: value 8.6V -> 8.7V
- L3: value L -> 27nH
- R27, R29, R31, R33: value 51k -> 100k
- R28, R30, R32, R34: value 10k -> 27k
- R42: value 0 -> 10
- moved R17 20.4 mm to (211.9, 70.9)
- moved LS1 8.02 mm to (207.4, 61.9), turned to 90 degrees
- moved C41 4.13 mm to (188.2, 62.4), turned to 0 degrees
- moved CR1 3.40 mm to (187.3, 66.9), turned to 0 degrees
- moved R8 2.65 mm to (180.4, 56.5), turned to 0 degrees
- moved R43 2.50 mm to (193.9, 70.9)
- moved U6 1.52 mm to (184.4, 57.1)
- moved R7 1.06 mm to (209.8, 86.0)
- moved C10 1.06 mm to (201.4, 77.5)
- moved C12 1.06 mm to (202.4, 78.5)
- moved C5 1.06 mm to (203.5, 79.6)
- moved R46 1.06 mm to (206.6, 82.8)
- moved R47 1.06 mm to (205.6, 81.7)
- moved R48 1.06 mm to (204.5, 80.7)
- moved C42 1.00 mm to (198.4, 70.9)
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Connections:
- Q4 pad 1: GND -> /pyro 2 drain
- Q4 pad 2: GND -> /pyro 2 drain
- Q4 pad 4: /pyro 2 drain -> GND
- Q4 pad 5: GND -> /pyro 2 drain
- Q4 pad 6: GND -> /pyro 2 drain
- Q4 pad D1: GND -> /pyro 2 drain
- Q4 pad D2: /pyro 2 drain -> GND
- Q5 pad 1: GND -> /pyro 3 drain
- Q5 pad 2: GND -> /pyro 3 drain
- Q5 pad 4: /pyro 3 drain -> GND
- Q5 pad 5: GND -> /pyro 3 drain
- Q5 pad 6: GND -> /pyro 3 drain
- Q5 pad D1: GND -> /pyro 3 drain
- Q5 pad D2: /pyro 3 drain -> GND
- Q6 pad 1: GND -> /pyro 4 drain
- Q6 pad 2: GND -> /pyro 4 drain
- Q6 pad 4: /pyro 4 drain -> GND
- Q6 pad 5: GND -> /pyro 4 drain
- Q6 pad 6: GND -> /pyro 4 drain
- Q6 pad D1: GND -> /pyro 4 drain
- Q6 pad D2: /pyro 4 drain -> GND
- R8 pad 1: +VBAT -> +VBAT safe
- U1 pad 14: unconnected-(U1-GPIO15-Pad14) -> /ADXL375 CS
- U1 pad 16: unconnected-(U1-GPIO16-Pad16) -> /BMP581 CS
- U1 pad 17: unconnected-(U1-GPIO17-Pad17) -> /SCK
- U1 pad 18: unconnected-(U1-GPIO18-Pad18) -> /BNO086 CS
- U1 pad 19: unconnected-(U1-GPIO19-Pad19) -> /MOSI
- U1 pad 20: unconnected-(U1-GPIO20-Pad20) -> /MISO
- U6 pad 1: +VBAT -> +VBAT safe
- U6 pad 2: +VBAT -> +VBAT safe
- U6 pad 3: +VBAT -> +VBAT safe
Routing:
- net +5V: track 40.0 -> 106.2 mm, vias 2 -> 3
- net /MOSI: track 14.1 -> 78.9 mm, vias 2 -> 4
- net /MISO: track 14.9 -> 77.5 mm, vias 3 -> 5
- net /MAX M10S boot: track 47.2 -> 1.45 mm
- net /SCK: track 36.9 -> 76.5 mm, vias 2 -> 4
- net /MAX M10S reset: track 37.3 -> 1.55 mm
- net /MAX M10S int: track 37.2 -> 1.55 mm
- net /MAX M10S timepulse: track 37.0 -> 1.55 mm
- net /MAX M10S TX: track 36.9 -> 1.55 mm
- net /MAX M10S RX: track 36.8 -> 1.55 mm
- net Net-(Q3-G): track 29.4 -> 0.00 mm, vias 1 -> 0
- net /buzzer: track 24.0 -> 0.00 mm, vias 2 -> 0
- net Net-(Q4-G): track 24.5 -> 1.02 mm
- net Net-(Q5-G): track 19.5 -> 1.02 mm
- net /BNO086 CS: track 0.00 -> 13.7 mm
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- added copper zone on In1.Cu, net +1.1V
- added copper zone on In1.Cu, net +12V pyro
- added copper zone on F.Cu, net +5V
- added copper zone on B.Cu, net +VBAT safe
- removed copper zone on In2.Cu, net +1.1V
- removed copper zone on In2.Cu, net +12V pyro
- removed copper zone on F.Cu, net Net-(D5-A)
Other:
- board text added: "{ "ViaStitching": "0.2", "entire": { "HSpacing": "1", "VSpacing": "1", "HOffset": "0", "VOffset": "0", "Clearance": "0.2", "Randomize": false } }"

Commit message: Final PCB with silkscreen
Parts:
- removed LS1: CPT-1203-78-SMT-TR, Snapeda:XDCR_CPT-1203-78-SMT-TR
- removed R17: 1k, Resistor_SMD:R_0603_1608Metric_Pad0.98x0.95mm_HandSolder
- moved R53 20.3 mm to (201.4, 52.6)
- moved R50 16.1 mm to (201.4, 56.6)
- moved R51 11.9 mm to (201.4, 60.6)
- moved R52 7.70 mm to (201.4, 64.7)
Connections:
- S1 pad 4: unconnected-(S1-COM_2-Pad4) -> GND
- S2 pad 4: unconnected-(S2-COM_2-Pad4) -> GND
- U1 pad 11: /MAX M10S boot -> /MAX M10S RX
- U1 pad 12: /MAX M10S reset -> /MAX M10S TX
- U1 pad 13: unconnected-(U1-GPIO14-Pad13) -> /MAX M10S boot
- U1 pad 17: /SCK -> /BNO086 CS
- U1 pad 18: /BNO086 CS -> /SCK
- U1 pad 36: /buzzer -> unconnected-(U1-GPIO28-Pad36)
- U1 pad 6: /MAX M10S int -> unconnected-(U1-GPIO8-Pad6)
- U1 pad 7: /MAX M10S timepulse -> /MAX M10S reset
- U1 pad 8: /MAX M10S RX -> /MAX M10S int
- U1 pad 9: /MAX M10S TX -> /MAX M10S timepulse
- U4 pad 4: GND -> +3.3V
Routing:
- net /MAX M10S boot: track 1.45 -> 48.2 mm
- net /MAX M10S reset: track 1.55 -> 39.3 mm
- net Net-(Q7-G): track 1.02 -> 38.1 mm
- net /MAX M10S TX: track 1.55 -> 37.8 mm
- net /MAX M10S int: track 1.55 -> 37.7 mm
- net /MAX M10S timepulse: track 1.55 -> 37.5 mm
- net /MAX M10S RX: track 1.55 -> 37.4 mm
- net Net-(Q4-G): track 1.02 -> 33.2 mm
- net Net-(Q5-G): track 1.02 -> 28.3 mm
- net Net-(Q6-G): track 1.02 -> 23.3 mm
- net Net-(LED2-DOUT): track 0.00 -> 12.5 mm
- net Net-(LED1-DOUT): track 0.00 -> 12.5 mm
- net Net-(LED3-DOUT): track 0.00 -> 9.06 mm
- net /pyro 4 gate: track 0.00 -> 6.36 mm, vias 0 -> 1
- net /pyro 3 gate: track 0.00 -> 5.70 mm, vias 0 -> 1
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Other:
- board text added: "+"
- board text added: "-"
- board text added: "12V"
- board text added: "3V"
- board text added: "5V"
- board text added: "A"
- board text added: "ARM"
- board text added: "B"
- board text added: "BAT"
- board text added: "IO1"
- board text added: "IO2"
- board text added: "K E R B"
- board text added: "MA"
- board text added: "MB"
- board text added: "PY1"
- board text added: "PY2"
- board text added: "PY3"
- board text added: "PY4"
- board text added: "REV 1.0"
- board text added: "S"
- board text added: "S1"
- board text added: "S2"
- board text added: "S3"
- board text added: "S4"
- board text added: "SW"
