File: flight computer/flight computer.kicad_pcb (KiCad board)
At the start: 4 copper layers, 43.2 x 99.1 mm, 158 parts, among them IC1 AT25SF128A-SHB-T, IC2 114993390, IC3 ADXL375BCCZ-RL, J1 JST, J10 Micro_SD_Card, J11 pyro 1, J12 pyro 2, J13 pyro 3, J14 pyro 4, J15 motor out, J16 5V out, J17 motor in, J18 servo 1, J19 servo 2, J2 battery in, J20 servo 3, J21 servo 4, J22 SMA-J-P-H-ST-EM1, J23 SMA-J-P-H-ST-EM1, J3 battery sw, J4 pyro sw, J5 12V out, J6 5V out, J7 3.3V out, J8 USB_C_Receptacle_USB2.0_16P, J9 GPIO, Q4 SIA440DJ-T1-GE3, Q5 SIA440DJ-T1-GE3, Q6 SIA440DJ-T1-GE3, Q7 SIA440DJ-T1-GE3, U1 RP2350B, U10 MAX-M10S-00B, U11 SISS65DN-T1-GE3, U4 AZ1117CH-3.3TRG1, U5 TPS56A37RPAR, U6 SISS65DN-T1-GE3, U7 BTM9011EP, U8 BMP581, U9 BNO086, Y1 ABM8-272-T3

Commit message: Generated Gerber Files
Connections:
- J16 pad 1: +5V -> +3.3V
Routing:
- net +5V: track 106.5 -> 91.4 mm
- net +3.3V: track 22.2 -> 37.1 mm, vias 17 -> 18
Changed lines of the file:
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@@
 		(capping no)
 		(filling no)
-		(zone_defaults)
 		(grid_origin 198.38 88.9)
 		(pcbplotparams
@@
 			(layers "*.Cu" "*.Mask")
 			(remove_unused_layers no)
-			(net "+5V")
+			(net "+3.3V")
 			(pinfunction "1_1")
 			(pintype "passive")
@@
 	)
 	(segment
-		(start 195.530689 107.95)
-		(end 195.880687 108.299998)
-		(width 0.2)
-		(layer "In1.Cu")
-		(net "+5V")
-	)
-	(segment
 		(start 192.480689 104.9)
 		(end 180.385 104.9)
@@
 	)
 	(segment
-		(start 180.84 107.95)
-		(end 195.530689 107.95)
-		(width 0.2)
-		(layer "In1.Cu")
-		(net "+5V")
-	)
-	(segment
 		(start 178.38 70.4)
 		(end 183.13 65.65)
@@
 	)
 	(via
+		(at 182.88 93.9)
+		(size 0.6)
+		(drill 0.3)
+		(layers "F.Cu" "B.Cu")
+		(free yes)
+		(net "+3.3V")
+	)
+	(via
 		(at 200.38 86.9)
 		(size 0.6)
@@
 		(net "+3.3V")
 	)
+	(segment
+		(start 182.88 105.91)
+		(end 180.84 107.95)
+		(width 0.2)
+		(layer "In2.Cu")
+		(net "+3.3V")
+	)
+	(segment
+		(start 182.88 93.9)
+		(end 182.88 105.91)
+		(width 0.2)
+		(layer "In2.Cu")
+		(net "+3.3V")
+	)
